Commit message: V1.2.0: - added limited joint trajectories; - updated/added robots and models; - updated tutorials; - bugfixes; - unified line-endings;

File: src/robotblockset/urdf_models/panda/panda.urdf (robot description, URDF)
Before this commit: robot panda, 13 links, 12 joints
Links:
- link panda_link6: geometry collision mesh filename=package://panda/meshes/collision/link6.obj; visual mesh filename=package://panda/meshes/visual/link6.dae
